File: Driver.kicad_sch (KiCad schematic)
At the start: 44 parts, among them Q1 SQJ886EP-T1_GE3, Q3 SQJ886EP-T1_GE3, Q5 SQJ886EP-T1_GE3, Q7 SQJ886EP-T1_GE3, U1 UCC21520DW, U4 UCC21520DW

Commit message: release prot.1 v0.1.0
Parts:
- Q1, Q5: footprint Package_SO:PowerPAK_SO-8L_Single -> Package_SO:PowerPAK_SO-8_Single
- Q3, Q7: footprint Package_SO:PowerPAK_SO-8L_Single -> RDC_footprint:PowerPAK_SO-8_Single_ThermalVias
Changed lines of the file:
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@@
       (effects (font (size 1.27 1.27)) (justify right))
     )
-    (property "Footprint" "Package_SO:PowerPAK_SO-8L_Single" (at 129.54 118.11 0)
+    (property "Footprint" "RDC_footprint:PowerPAK_SO-8_Single_ThermalVias" (at 129.54 118.11 0)
       (effects (font (size 1.27 1.27)) hide)
     )
@@
       (effects (font (size 1.27 1.27)) (justify right))
     )
-    (property "Footprint" "Package_SO:PowerPAK_SO-8L_Single" (at 168.91 118.11 0)
+    (property "Footprint" "RDC_footprint:PowerPAK_SO-8_Single_ThermalVias" (at 168.91 118.11 0)
       (effects (font (size 1.27 1.27)) hide)
     )
@@
       (effects (font (size 1.27 1.27)) (justify right))
     )
-    (property "Footprint" "Package_SO:PowerPAK_SO-8L_Single" (at 129.54 96.52 0)
+    (property "Footprint" "Package_SO:PowerPAK_SO-8_Single" (at 129.54 96.52 0)
       (effects (font (size 1.27 1.27)) hide)
     )
@@
       (effects (font (size 1.27 1.27)) (justify right))
     )
-    (property "Footprint" "Package_SO:PowerPAK_SO-8L_Single" (at 168.91 96.52 0)
-      (effects (font (size 1.27 1.27)) hide)
-    )
+    (property "Footprint" "Package_SO:PowerPAK_SO-8_Single" (at 168.91 96.52 0)
+      (effects (font (size 1.27 1.27)) hide)
+    )

Commit message: Update PCB design & add microSD connector
Parts:
- C24: renamed from C51; footprint Capacitor_SMD:C_0603_1608Metric_Pad1.08x0.95mm_HandSolder -> Capacitor_SMD:C_0402_1005Metric
- C25: renamed from C53; footprint Capacitor_SMD:C_0603_1608Metric_Pad1.08x0.95mm_HandSolder -> Capacitor_SMD:C_0402_1005Metric
- C26: renamed from C49; footprint Capacitor_SMD:C_0402_1005Metric_Pad0.74x0.62mm_HandSolder -> Capacitor_SMD:C_0402_1005Metric
- C27: footprint Capacitor_SMD:C_0402_1005Metric_Pad0.74x0.62mm_HandSolder -> Capacitor_SMD:C_0402_1005Metric
- C28: renamed from C16; footprint Capacitor_SMD:C_0402_1005Metric_Pad0.74x0.62mm_HandSolder -> Capacitor_SMD:C_0402_1005Metric
- C29: renamed from C18; footprint Capacitor_SMD:C_1210_3225Metric_Pad1.33x2.70mm_HandSolder -> Capacitor_SMD:C_1210_3225Metric
- C30: renamed from C17; footprint Capacitor_SMD:C_1210_3225Metric_Pad1.33x2.70mm_HandSolder -> Capacitor_SMD:C_1210_3225Metric
- C31: renamed from C15; footprint Capacitor_SMD:C_1210_3225Metric_Pad1.33x2.70mm_HandSolder -> Capacitor_SMD:C_1210_3225Metric
- C32: renamed from C19; footprint Capacitor_SMD:C_1210_3225Metric_Pad1.33x2.70mm_HandSolder -> Capacitor_SMD:C_1210_3225Metric
- C33: renamed from C14; footprint Capacitor_SMD:C_0402_1005Metric_Pad0.74x0.62mm_HandSolder -> Capacitor_SMD:C_0402_1005Metric
- C34: renamed from C45; footprint Capacitor_SMD:C_0402_1005Metric_Pad0.74x0.62mm_HandSolder -> Capacitor_SMD:C_0402_1005Metric
- C35: renamed from C47; footprint Capacitor_SMD:C_0402_1005Metric_Pad0.74x0.62mm_HandSolder -> Capacitor_SMD:C_0402_1005Metric
- C36: renamed from C56; footprint Capacitor_SMD:C_0603_1608Metric_Pad1.08x0.95mm_HandSolder -> Capacitor_SMD:C_0402_1005Metric
- C37: renamed from C55; footprint Capacitor_SMD:C_0603_1608Metric_Pad1.08x0.95mm_HandSolder -> Capacitor_SMD:C_0402_1005Metric
- Q1: footprint Package_SO:PowerPAK_SO-8_Single -> RDC_footprint:PowerPAK_SO-8_Single_ThermalVias
- Q2: renamed from Q3; footprint RDC_footprint:PowerPAK_SO-8_Single_ThermalVias -> Package_SO:PowerPAK_SO-8_Single
- Q3: renamed from Q5; footprint Package_SO:PowerPAK_SO-8_Single -> RDC_footprint:PowerPAK_SO-8_Single_ThermalVias
- Q4: renamed from Q7; footprint RDC_footprint:PowerPAK_SO-8_Single_ThermalVias -> Package_SO:PowerPAK_SO-8_Single
- R13: renamed from R38; footprint Resistor_SMD:R_0603_1608Metric_Pad0.98x0.95mm_HandSolder -> Capacitor_SMD:C_0402_1005Metric
- R14: renamed from R36; footprint Resistor_SMD:R_0603_1608Metric_Pad0.98x0.95mm_HandSolder -> Capacitor_SMD:C_0402_1005Metric
- R15: renamed from R20; footprint Resistor_SMD:R_0402_1005Metric_Pad0.72x0.64mm_HandSolder -> Resistor_SMD:R_0402_1005Metric
- R16: renamed from R32; footprint Resistor_SMD:R_0402_1005Metric_Pad0.72x0.64mm_HandSolder -> Resistor_SMD:R_0402_1005Metric
- R17: renamed from R4; footprint Resistor_SMD:R_1206_3216Metric_Pad1.30x1.75mm_HandSolder -> Resistor_SMD:R_1206_3216Metric
- R18: renamed from R2; footprint Resistor_SMD:R_0805_2012Metric_Pad1.20x1.40mm_HandSolder -> Resistor_SMD:R_0805_2012Metric
- R19: renamed from R3; footprint Resistor_SMD:R_0805_2012Metric_Pad1.20x1.40mm_HandSolder -> Resistor_SMD:R_0805_2012Metric
- R20: renamed from R24; footprint Resistor_SMD:R_0402_1005Metric_Pad0.72x0.64mm_HandSolder -> Resistor_SMD:R_0402_1005Metric
- R21: renamed from R26; footprint Resistor_SMD:R_0402_1005Metric_Pad0.72x0.64mm_HandSolder -> Resistor_SMD:R_0402_1005Metric
- R22: renamed from R28; footprint Resistor_SMD:R_0402_1005Metric_Pad0.72x0.64mm_HandSolder -> Resistor_SMD:R_0402_1005Metric
- R23: renamed from R30; footprint Resistor_SMD:R_0402_1005Metric_Pad0.72x0.64mm_HandSolder -> Resistor_SMD:R_0402_1005Metric
- R24: renamed from R6; footprint Resistor_SMD:R_0805_2012Metric_Pad1.20x1.40mm_HandSolder -> Resistor_SMD:R_0805_2012Metric
- R25: renamed from R7; footprint Resistor_SMD:R_0805_2012Metric_Pad1.20x1.40mm_HandSolder -> Resistor_SMD:R_0805_2012Metric
- R26: renamed from R5; footprint Resistor_SMD:R_1206_3216Metric_Pad1.30x1.75mm_HandSolder -> Resistor_SMD:R_1206_3216Metric
- R27: renamed from R34; footprint Resistor_SMD:R_0402_1005Metric_Pad0.72x0.64mm_HandSolder -> Resistor_SMD:R_0402_1005Metric
- R28: renamed from R22; footprint Resistor_SMD:R_0402_1005Metric_Pad0.72x0.64mm_HandSolder -> Resistor_SMD:R_0402_1005Metric
- R29: renamed from R41; footprint Resistor_SMD:R_0603_1608Metric_Pad0.98x0.95mm_HandSolder -> Capacitor_SMD:C_0402_1005Metric
- R30: renamed from R40; footprint Resistor_SMD:R_0603_1608Metric_Pad0.98x0.95mm_HandSolder -> Capacitor_SMD:C_0402_1005Metric
- renumbered D14 to D10, D2 to D11, D1 to D6, D9 to D7, D13 to D8, D11 to D9, U1 to U4, U4 to U5
Other:
- moved on the sheet: D10, D7, D8, D9

Commit message: update BOM
Parts:
- removed R15, R28: 10k, Resistor_SMD:R_0402_1005Metric, symbol Device:R
- C26: renamed from C24; LCSC (none) -> C1562
- C27: renamed from C25; LCSC (none) -> C1562
- C28: renamed from C26; value 22nF -> 0.1uF; LCSC (none) -> C307331
- C29: renamed from C27; value 1nF -> 0.1uF; LCSC (none) -> C307331
- C30: renamed from C28; value 0.1u -> 0.1uF; LCSC (none) -> C307331
- C31: renamed from C29; value 10u -> 10uF; LCSC (none) -> C77102
- C32: renamed from C30; value 10u -> 10uF; LCSC (none) -> C77102
- C33: renamed from C31; value 10u -> 10uF; LCSC (none) -> C77102
- C34: renamed from C32; value 10u -> 10uF; LCSC (none) -> C77102
- C35: renamed from C33; value 0.1u -> 0.1uF; LCSC (none) -> C307331
- C36: renamed from C34; value 1nF -> 0.1uF; LCSC (none) -> C307331
- C37: renamed from C35; value 22nF -> 0.1uF; LCSC (none) -> C307331
- C38: renamed from C36; LCSC (none) -> C1562
- C39: renamed from C37; LCSC (none) -> C1562
- D10, D11, D6, D7, D8, D9: LCSC (none) -> C509937
- Q2: renamed from Q1; footprint RDC_footprint:PowerPAK_SO-8_Single_ThermalVias -> RDC_footprint:Infineon_PG-TDSON-8_6.15x5.15mm_thermalvia; FT Rotation Offset (none) -> -90; LCSC (none) -> C501507
- Q3: renamed from Q2; footprint Package_SO:PowerPAK_SO-8_Single -> Package_SON:Infineon_PG-TDSON-8_6.15x5.15mm; FT Rotation Offset (none) -> -90; LCSC (none) -> C501507
- Q4: renamed from Q3; footprint RDC_footprint:PowerPAK_SO-8_Single_ThermalVias -> RDC_footprint:Infineon_PG-TDSON-8_6.15x5.15mm_thermalvia; FT Rotation Offset (none) -> -90; LCSC (none) -> C501507
- Q5: renamed from Q4; footprint Package_SO:PowerPAK_SO-8_Single -> Package_SON:Infineon_PG-TDSON-8_6.15x5.15mm; FT Rotation Offset (none) -> -90; LCSC (none) -> C501507
- R28: renamed from R13; footprint Capacitor_SMD:C_0402_1005Metric -> Resistor_SMD:R_0402_1005Metric; LCSC (none) -> C25125
- R29: renamed from R14; footprint Capacitor_SMD:C_0402_1005Metric -> Resistor_SMD:R_0402_1005Metric; LCSC (none) -> C25125
- R30: renamed from R16; LCSC (none) -> C25765
- R31: renamed from R17; LCSC (none) -> C25334
- R32: renamed from R18; LCSC (none) -> C17415
- R33: renamed from R19; LCSC (none) -> C17415
- R34: renamed from R20; LCSC (none) -> C25765
- R35: renamed from R21; LCSC (none) -> C25765
- R36: renamed from R22; LCSC (none) -> C25765
- R37: renamed from R23; LCSC (none) -> C25765
- R38: renamed from R24; LCSC (none) -> C17415
- R39: renamed from R25; LCSC (none) -> C17415
- R40: renamed from R26; LCSC (none) -> C25334
- R41: renamed from R27; LCSC (none) -> C25765
- R42: renamed from R29; footprint Capacitor_SMD:C_0402_1005Metric -> Resistor_SMD:R_0402_1005Metric; LCSC (none) -> C25125
- R43: renamed from R30; footprint Capacitor_SMD:C_0402_1005Metric -> Resistor_SMD:R_0402_1005Metric; LCSC (none) -> C25125
- U4, U5: FT Rotation Offset (none) -> -90; LCSC (none) -> C601651
Other:
- moved on the sheet: C26, C27, C38, C39, R28, R29, R42, R43
