File: STM32F405.kicad_sch (KiCad schematic)
At the start: 22 parts, among them SW1 SW_Push, SW3 SW_Push, U3 STM32F405RGTx, Y1 25MHz

Commit message: update BOM
Parts:
- C13: renamed from C11; value 0.1u -> 0.1uF; LCSC (none) -> C307331
- C14: renamed from C12; LCSC (none) -> C1549
- C15: renamed from C13; LCSC (none) -> C1549
- C16: renamed from C14; LCSC (none) -> C23630
- C17: renamed from C15; LCSC (none) -> C23630
- C18: renamed from C16; value 0.1u -> 0.1uF; LCSC (none) -> C307331
- C19: renamed from C17; LCSC (none) -> C23733
- C20: renamed from C18; LCSC (none) -> C52923
- C21: renamed from C19; value 0.1u -> 0.1uF; LCSC (none) -> C307331
- C22: renamed from C20; value 0.1u -> 0.1uF; LCSC (none) -> C307331
- C23: renamed from C21; value 0.1u -> 0.1uF; LCSC (none) -> C307331
- C24: renamed from C22; value 0.1u -> 0.1uF; LCSC (none) -> C307331
- C25: renamed from C23; value 0.1u -> 0.1uF; LCSC (none) -> C307331
- D6: LCSC (none) -> C2296
- L1: LCSC (none) -> C1017
- R16: LCSC (none) -> C23138
- R25: renamed from R7; LCSC (none) -> C25744
- R26: renamed from R67; LCSC (none) -> C25744
- Y1: LCSC (none) -> C9006
- renumbered SW1 to SW3, SW3 to SW4
