File: 24-12V_StepDown_DCDC.kicad_sch (KiCad schematic)
At the start: 8 parts, among them U10 TPS5430DDA

Commit message: Modified DCDC converter coil
Parts:
- L2: footprint Inductor_SMD:L_Changjiang_FNR4020S -> Inductor_SMD:L_Sunlord_SWPA5040S
Changed lines of the file:
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@@
       (effects (font (size 1.27 1.27)))
     )
-    (property "Footprint" "Inductor_SMD:L_Changjiang_FNR4020S" (at 162.56 87.63 0)
+    (property "Footprint" "Inductor_SMD:L_Sunlord_SWPA5040S" (at 162.56 87.63 0)
       (effects (font (size 1.27 1.27)) hide)
     )

Commit message: update BOM
Parts:
- C1: value 220u -> 220uF
- C52: value 10u -> 10uF; footprint Capacitor_SMD:C_0603_1608Metric -> Capacitor_SMD:C_0805_2012Metric; LCSC (none) -> C440198
- C54: value 0.01u -> 0.01uF; LCSC (none) -> C57112
- D19: LCSC (none) -> C509937
- L2: LCSC (none) -> C44888
- R1: LCSC (none) -> C4109
- R1: LCSC (none) -> C25762
- U10: LCSC (none) -> C9864
Changed lines of the file:
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@@
       (effects (font (size 1.27 1.27)) (justify right))
     )
-    (property "Value" "0.01u" (at 144.78 78.74 90)
+    (property "Value" "0.01uF" (at 144.78 78.74 90)
       (effects (font (size 1.27 1.27)) (justify right))
     )
@@
       (effects (font (size 1.27 1.27)) hide)
     )
+    (property "LCSC" "C57112" (at 147.32 82.55 0)
+      (effects (font (size 1.27 1.27)) hide)
+    )
+    (property "FT Rotation Offset" "" (at 147.32 82.55 0)
+      (effects (font (size 1.27 1.27)) hide)
+    )
     (pin "1")
     (pin "2")
@@
         )
         (path "/3152684b-d11f-4a9a-8e6c-09965044adbd/796ce04a-783e-4174-adea-a6f6cdf2f836"
-          (reference "C56") (unit 1)
+          (reference "C60") (unit 1)
         )
       )
@@
       (effects (font (size 1.27 1.27)) hide)
     )
+    (property "LCSC" "C44888" (at 162.56 87.63 0)
+      (effects (font (size 1.27 1.27)) hide)
+    )
+    (property "FT Rotation Offset" "" (at 162.56 87.63 0)
+      (effects (font (size 1.27 1.27)) hide)
+    )
     (pin "1")
     (pin "2")
@@
       (effects (font (size 1.27 1.27)) (justify right))
     )
-    (property "Value" "10u" (at 100.33 91.44 0)
-      (effects (font (size 1.27 1.27)) (justify right))
-    )
-    (property "Footprint" "Capacitor_SMD:C_0603_1608Metric" (at 101.6 88.9 0)
+    (property "Value" "10uF" (at 100.33 91.44 0)
+      (effects (font (size 1.27 1.27)) (justify right))
+    )
+    (property "Footprint" "Capacitor_SMD:C_0805_2012Metric" (at 101.6 88.9 0)
       (effects (font (size 1.27 1.27)) hide)
     )
@@
       (effects (font (size 1.27 1.27)) hide)
     )
+    (property "LCSC" "C440198" (at 101.6 88.9 0)
+      (effects (font (size 1.27 1.27)) hide)
+    )
+    (property "FT Rotation Offset" "" (at 101.6 88.9 0)
+      (effects (font (size 1.27 1.27)) hide)
+    )
     (pin "1")
     (pin "2")
@@
         )
         (path "/3152684b-d11f-4a9a-8e6c-09965044adbd/796ce04a-783e-4174-adea-a6f6cdf2f836"
-          (reference "C55") (unit 1)
+          (reference "C59") (unit 1)
         )
       )
@@
       (effects (font (size 1.27 1.27)) hide)
     )
+    (property "LCSC" "C509937" (at 154.94 93.98 0)
+      (effects (font (size 1.27 1.27)) hide)
+    )
+    (property "FT Rotation Offset" "" (at 154.94 93.98 0)
+      (effects (font (size 1.27 1.27)) hide)
+    )
     (pin "1")
     (pin "2")
@@
       (effects (font (size 1.27 1.27)) (justify left))
     )
-    (property "Value" "220u" (at 175.26 95.25 0)
+    (property "Value" "220uF" (at 175.26 95.25 0)
       (effects (font (size 1.27 1.27)) (justify left))
     )
@@
     )
     (property "Datasheet" "~" (at 171.45 93.98 0)
+      (effects (font (size 1.27 1.27)) hide)
+    )
+    (property "LCSC" "" (at 171.45 93.98 0)
+      (effects (font (size 1.27 1.27)) hide)
+    )
+    (property "FT Rotation Offset" "" (at 171.45 93.98 0)
       (effects (font (size 1.27 1.27)) hide)
     )
@@
       (effects (font (size 1.27 1.27)) hide)
     )
+    (property "LCSC" "C4109" (at 185.42 104.14 0)
+      (effects (font (size 1.27 1.27)) hide)
+    )
+    (property "FT Rotation Offset" "" (at 185.42 104.14 0)
+      (effects (font (size 1.27 1.27)) hide)
+    )
     (pin "1")
     (pin "2")
@@
         )
         (path "/3152684b-d11f-4a9a-8e6c-09965044adbd/796ce04a-783e-4174-adea-a6f6cdf2f836"
-          (reference "R65") (unit 1)
+          (reference "R63") (unit 1)
         )
       )
@@
     )
     (property "Datasheet" "~" (at 185.42 93.98 0)
+      (effects (font (size 1.27 1.27)) hide)
+    )
+    (property "LCSC" "C25762" (at 185.42 93.98 0)
+      (effects (font (size 1.27 1.27)) hide)
+    )
+    (property "FT Rotation Offset" "" (at 185.42 93.98 0)
       (effects (font (size 1.27 1.27)) hide)
     )
@@
         )
         (path "/3152684b-d11f-4a9a-8e6c-09965044adbd/796ce04a-783e-4174-adea-a6f6cdf2f836"
-          (reference "R64") (unit 1)
+          (reference "R62") (unit 1)
         )
       )
@@
     )
     (property "Datasheet" "http://www.ti.com/lit/ds/symlink/tps5430.pdf" (at 132.08 87.63 0)
+      (effects (font (size 1.27 1.27)) hide)
+    )
+    (property "LCSC" "C9864" (at 132.08 87.63 0)
+      (effects (font (size 1.27 1.27)) hide)
+    )
+    (property "FT Rotation Offset" "" (at 132.08 87.63 0)
       (effects (font (size 1.27 1.27)) hide)
     )
@@
         )
         (path "/3152684b-d11f-4a9a-8e6c-09965044adbd/796ce04a-783e-4174-adea-a6f6cdf2f836"
-          (reference "U8") (unit 1)
-        )
-      )
+          (reference "U10") (unit 1)
+        )
+      )

Commit message: Board for ordering
Parts:
- added R4: 10k, Resistor_SMD:R_1206_3216Metric, symbol Device:R
- D19: LCSC C509937 -> C22466347
Connections:
- net GND: now also R4.2
- net Power_OUT: now also R4.1
Other:
- moved on the sheet: R1
Changed lines of the file:
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@@
   (junction (at 101.6 82.55) (diameter 0) (color 0 0 0 0)
   )
-  (junction (at 185.42 99.06) (diameter 0) (color 0 0 0 0)
+  (junction (at 187.96 99.06) (diameter 0) (color 0 0 0 0)
   )
   (junction (at 154.94 87.63) (diameter 0) (color 0 0 0 0)
   )
-  (junction (at 185.42 87.63) (diameter 0) (color 0 0 0 0)
+  (junction (at 198.12 87.63) (diameter 0) (color 0 0 0 0)
+  )
+  (junction (at 187.96 87.63) (diameter 0) (color 0 0 0 0)
   )
   (junction (at 129.54 100.33) (diameter 0) (color 0 0 0 0)
@@
   )
   (no_connect (at 119.38 92.71))
-  (wire (pts (xy 185.42 90.17) (xy 185.42 87.63))
+  (wire (pts (xy 198.12 87.63) (xy 198.12 95.25))
+    (stroke (width 0) (type default))
+  )
+  (wire (pts (xy 187.96 90.17) (xy 187.96 87.63))
     (stroke (width 0) (type default))
   )
@@
     (stroke (width 0) (type default))
   )
-  (wire (pts (xy 177.8 109.22) (xy 144.78 109.22))
-    (stroke (width 0) (type default))
-  )
-  (wire (pts (xy 185.42 87.63) (xy 201.93 87.63))
-    (stroke (width 0) (type default))
-  )
-  (wire (pts (xy 185.42 97.79) (xy 185.42 99.06))
+  (wire (pts (xy 180.34 109.22) (xy 144.78 109.22))
+    (stroke (width 0) (type default))
+  )
+  (wire (pts (xy 171.45 87.63) (xy 187.96 87.63))
+    (stroke (width 0) (type default))
+  )
+  (wire (pts (xy 187.96 97.79) (xy 187.96 99.06))
+    (stroke (width 0) (type default))
+  )
+  (wire (pts (xy 187.96 87.63) (xy 198.12 87.63))
     (stroke (width 0) (type default))
   )
@@
     (stroke (width 0) (type default))
   )
-  (wire (pts (xy 185.42 107.95) (xy 185.42 113.03))
-    (stroke (width 0) (type default))
-  )
-  (wire (pts (xy 177.8 109.22) (xy 177.8 99.06))
+  (wire (pts (xy 187.96 107.95) (xy 187.96 113.03))
+    (stroke (width 0) (type default))
+  )
+  (wire (pts (xy 180.34 109.22) (xy 180.34 99.06))
     (stroke (width 0) (type default))
   )
@@
     (stroke (width 0) (type default))
   )
-  (wire (pts (xy 177.8 99.06) (xy 185.42 99.06))
+  (wire (pts (xy 198.12 102.87) (xy 198.12 113.03))
+    (stroke (width 0) (type default))
+  )
+  (wire (pts (xy 180.34 99.06) (xy 187.96 99.06))
+    (stroke (width 0) (type default))
+  )
+  (wire (pts (xy 198.12 87.63) (xy 201.93 87.63))
     (stroke (width 0) (type default))
   )
@@
     (stroke (width 0) (type default))
   )
-  (wire (pts (xy 171.45 87.63) (xy 185.42 87.63))
-    (stroke (width 0) (type default))
-  )
   (wire (pts (xy 132.08 97.79) (xy 132.08 100.33))
     (stroke (width 0) (type default))
@@
     (stroke (width 0) (type default))
   )
-  (wire (pts (xy 185.42 99.06) (xy 185.42 100.33))
+  (wire (pts (xy 187.96 99.06) (xy 187.96 100.33))
     (stroke (width 0) (type default))
   )
@@
     (effects (font (size 1.27 1.27)) (justify right))
   )
-  (hierarchical_label "GND" (shape output) (at 185.42 113.03 270) (fields_autoplaced)
+  (hierarchical_label "GND" (shape output) (at 187.96 113.03 270) (fields_autoplaced)
     (effects (font (size 1.27 1.27)) (justify right))
   )
@@
     (effects (font (size 1.27 1.27)) (justify left))
   )
+  (hierarchical_label "GND" (shape output) (at 198.12 113.03 270) (fields_autoplaced)
+    (effects (font (size 1.27 1.27)) (justify right))
+  )
   (hierarchical_label "GND" (shape output) (at 154.94 100.33 270) (fields_autoplaced)
     (effects (font (size 1.27 1.27)) (justify right))
@@
         (path "/3152684b-d11f-4a9a-8e6c-09965044adbd/796ce04a-783e-4174-adea-a6f6cdf2f836"
           (reference "C59") (unit 1)
+        )
+      )
+    )
+  )
+  (symbol (lib_id "Device:R") (at 198.12 99.06 0) (unit 1)
+    (in_bom yes) (on_board yes) (dnp no)
+    (property "Reference" "R4" (at 196.85 97.79 0)
+      (effects (font (size 1.27 1.27)) (justify right))
+    )
+    (property "Value" "10k" (at 196.85 100.33 0)
+      (effects (font (size 1.27 1.27)) (justify right))
+    )
+    (property "Footprint" "Resistor_SMD:R_1206_3216Metric" (at 196.342 99.06 90)
+      (effects (font (size 1.27 1.27)) hide)
+    )
+    (property "Datasheet" "~" (at 198.12 99.06 0)
+      (effects (font (size 1.27 1.27)) hide)
+    )
+    (property "LCSC" "C17902" (at 198.12 99.06 0)
+      (effects (font (size 1.27 1.27)) hide)
+    )
+    (property "FT Rotation Offset" "" (at 198.12 99.06 0)
+      (effects (font (size 1.27 1.27)) hide)
+    )
+    (pin "1")
+    (pin "2")
+    (instances
+      (project "schematic_MD"
+        (path "/3152684b-d11f-4a9a-8e6c-09965044adbd"
+          (reference "R4") (unit 1)
+        )
+        (path "/3152684b-d11f-4a9a-8e6c-09965044adbd/2d267caf-42fc-44ea-97db-65c2b77a1587"
+          (reference "R70") (unit 1)
+        )
+        (path "/3152684b-d11f-4a9a-8e6c-09965044adbd/796ce04a-783e-4174-adea-a6f6cdf2f836"
+          (reference "R71") (unit 1)
         )
       )
@@
       (effects (font (size 1.27 1.27)) hide)
     )
-    (property "LCSC" "C509937" (at 154.94 93.98 0)
+    (property "LCSC" "C22466347" (at 154.94 93.98 0)
       (effects (font (size 1.27 1.27)) hide)
     )
@@
     )
   )
-  (symbol (lib_id "Device:R") (at 185.42 104.14 0) (unit 1)
-    (in_bom yes) (on_board yes) (dnp no)
-    (property "Reference" "R1" (at 184.15 102.87 0)
-      (effects (font (size 1.27 1.27)) (justify right))
-    )
-    (property "Value" "2k" (at 184.15 105.41 0)
-      (effects (font (size 1.27 1.27)) (justify right))
-    )
-    (property "Footprint" "Resistor_SMD:R_0402_1005Metric" (at 183.642 104.14 90)
-      (effects (font (size 1.27 1.27)) hide)
-    )
-    (property "Datasheet" "~" (at 185.42 104.14 0)
-      (effects (font (size 1.27 1.27)) hide)
-    )
-    (property "LCSC" "C4109" (at 185.42 104.14 0)
-      (effects (font (size 1.27 1.27)) hide)
-    )
-    (property "FT Rotation Offset" "" (at 185.42 104.14 0)
+  (symbol (lib_id "Device:R") (at 187.96 104.14 0) (unit 1)
+    (in_bom yes) (on_board yes) (dnp no)
+    (property "Reference" "R1" (at 186.69 102.87 0)
+      (effects (font (size 1.27 1.27)) (justify right))
+    )
+    (property "Value" "2k" (at 186.69 105.41 0)
+      (effects (font (size 1.27 1.27)) (justify right))
+    )
+    (property "Footprint" "Resistor_SMD:R_0402_1005Metric" (at 186.182 104.14 90)
+      (effects (font (size 1.27 1.27)) hide)
+    )
+    (property "Datasheet" "~" (at 187.96 104.14 0)
+      (effects (font (size 1.27 1.27)) hide)
+    )
+    (property "LCSC" "C4109" (at 187.96 104.14 0)
+      (effects (font (size 1.27 1.27)) hide)
+    )
+    (property "FT Rotation Offset" "" (at 187.96 104.14 0)
       (effects (font (size 1.27 1.27)) hide)
     )
@@
     )
   )
-  (symbol (lib_id "Device:R") (at 185.42 93.98 0) (unit 1)
-    (in_bom yes) (on_board yes) (dnp no)
-    (property "Reference" "R1" (at 184.15 92.71 0)
-      (effects (font (size 1.27 1.27)) (justify right))
-    )
-    (property "Value" "18k" (at 184.15 95.25 0)
-      (effects (font (size 1.27 1.27)) (justify right))
-    )
-    (property "Footprint" "Resistor_SMD:R_0402_1005Metric" (at 183.642 93.98 90)
-      (effects (font (size 1.27 1.27)) hide)
-    )
-    (property "Datasheet" "~" (at 185.42 93.98 0)
-      (effects (font (size 1.27 1.27)) hide)
-    )
-    (property "LCSC" "C25762" (at 185.42 93.98 0)
-      (effects (font (size 1.27 1.27)) hide)
-    )
-    (property "FT Rotation Offset" "" (at 185.42 93.98 0)
-      (effects (font (size 1.27 1.27)) hide)
-    )
+  (symbol (lib_id "Device:R") (at 187.96 93.98 0) (unit 1)
+    (in_bom yes) (on_board yes) (dnp no)
+    (property "Reference" "R1" (at 186.69 92.71 0)
+      (effects (font (size 1.27 1.27)) (justify right))
+    )
+    (property "Value" "18k" (at 186.69 95.25 0)
+      (effects (font (size 1.27 1.27)) (justify right))
+    )
+    (property "Footprint" "Resistor_SMD:R_0402_1005Metric" (at 186.182 93.98 90)
+      (effects (font (size 1.27 1.27)) hide)
+    )
+    (property "Datasheet" "~" (at 187.96 93.98 0)
+      (effects (font (size 1.27 1.27)) hide)
+    )
+    (property "LCSC" "C25762" (at 187.96 93.98 0)
+      (effects (font (size 1.27 1.27)) hide)
+    )
+    (property "FT Rotation Offset" "" (at 187.96 93.98 0)
+      (effects (font (size 1.27 1.27)) hide)
+    )
