File: Logic_power.kicad_sch (KiCad schematic)
At the start: 12 parts, among them U10 TPS5430DDA, U9 XC6206P332MR-G

Commit message: 制御回路完成
Parts:
- removed C53: 0.1u, Capacitor_SMD:C_0603_1608Metric, symbol Device:C_Small
- added C1: 220u, Capacitor_THT:CP_Radial_D8.0mm_P3.50mm, symbol Device:C_Polarized
- L2: footprint (none) -> Inductor_SMD:L_Changjiang_FNR4020S
- R1: footprint Resistor_SMD:R_0603_1608Metric -> Resistor_SMD:R_0402_1005Metric
Connections:
- net 5V_OUT: now also C1.1; no longer C54.2
- net GND: now also C1.2
- net at D19.1 (K), L2.1, U10.8 (PH): now also C54.2
Other:
- moved on the sheet: C54, C57, C58, D18, D19, L2, R1, U9

Commit message: Change GND plene
Parts:
- L2: footprint Inductor_SMD:L_Changjiang_FNR4020S -> Inductor_SMD:L_Sunlord_SWPA5040S
Changed lines of the file:
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@@
       (effects (font (size 1.27 1.27)))
     )
-    (property "Footprint" "Inductor_SMD:L_Changjiang_FNR4020S" (at 97.79 34.29 0)
+    (property "Footprint" "Inductor_SMD:L_Sunlord_SWPA5040S" (at 97.79 34.29 0)
       (effects (font (size 1.27 1.27)) hide)
     )
@@
       (effects (font (size 1.27 1.27)) hide)
     )
+    (pin "1")
+    (pin "2")
+    (pin "3")
+    (pin "4")
     (pin "5")
-    (pin "4")
+    (pin "6")
+    (pin "7")
     (pin "8")
-    (pin "7")
-    (pin "2")
     (pin "9")
-    (pin "1")
-    (pin "6")
-    (pin "3")
     (instances
       (project "schematic_MD"

Commit message: update BOM
Parts:
- C1: value 220u -> 220uF
- C54: renamed from C52; value 10u -> 10uF; footprint Capacitor_SMD:C_0603_1608Metric -> Capacitor_SMD:C_0805_2012Metric; LCSC (none) -> C440198
- C55: renamed from C54; value 0.01u -> 0.01uF; LCSC (none) -> C57112
- C57, C58: LCSC (none) -> C15849
- D18: renamed from D19; LCSC (none) -> C509937
- D19: renamed from D18; LCSC (none) -> C509937
- L2: LCSC (none) -> C44888
- R1: LCSC (none) -> C51721
- R1: LCSC (none) -> C25752
- U8: renamed from U10; LCSC (none) -> C9864
- U9: FT Rotation Offset (none) -> 180; LCSC (none) -> C5446
Changed lines of the file:
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@@
       (effects (font (size 1.27 1.27)) (justify left))
     )
-    (property "Value" "220u" (at 111.76 41.91 0)
+    (property "Value" "220uF" (at 111.76 41.91 0)
       (effects (font (size 1.27 1.27)) (justify left))
     )
@@
     )
     (property "Datasheet" "~" (at 107.95 40.64 0)
+      (effects (font (size 1.27 1.27)) hide)
+    )
+    (property "LCSC" "" (at 107.95 40.64 0)
+      (effects (font (size 1.27 1.27)) hide)
+    )
+    (property "FT Rotation Offset" "" (at 107.95 40.64 0)
       (effects (font (size 1.27 1.27)) hide)
     )
@@
         )
         (path "/3152684b-d11f-4a9a-8e6c-09965044adbd/2d267caf-42fc-44ea-97db-65c2b77a1587"
-          (reference "C53") (unit 1)
+          (reference "C56") (unit 1)
         )
       )
@@
   (symbol (lib_id "Device:C_Small") (at 83.82 29.21 90) (mirror x) (unit 1)
     (in_bom yes) (on_board yes) (dnp no)
-    (property "Reference" "C54" (at 81.28 22.86 90)
-      (effects (font (size 1.27 1.27)) (justify right))
-    )
-    (property "Value" "0.01u" (at 81.28 25.4 90)
+    (property "Reference" "C55" (at 81.28 22.86 90)
+      (effects (font (size 1.27 1.27)) (justify right))
+    )
+    (property "Value" "0.01uF" (at 81.28 25.4 90)
       (effects (font (size 1.27 1.27)) (justify right))
     )
@@
       (effects (font (size 1.27 1.27)) hide)
     )
-    (pin "1")
-    (pin "2")
-    (instances
-      (project "schematic_MD"
-        (path "/3152684b-d11f-4a9a-8e6c-09965044adbd/2d267caf-42fc-44ea-97db-65c2b77a1587"
-          (reference "C54") (unit 1)
+    (property "LCSC" "C57112" (at 83.82 29.21 0)
+      (effects (font (size 1.27 1.27)) hide)
+    )
+    (property "FT Rotation Offset" "" (at 83.82 29.21 0)
+      (effects (font (size 1.27 1.27)) hide)
+    )
+    (pin "1")
+    (pin "2")
+    (instances
+      (project "schematic_MD"
+        (path "/3152684b-d11f-4a9a-8e6c-09965044adbd/2d267caf-42fc-44ea-97db-65c2b77a1587"
+          (reference "C55") (unit 1)
         )
       )
@@
   (symbol (lib_id "Device:D_Schottky") (at 91.44 40.64 270) (unit 1)
     (in_bom yes) (on_board yes) (dnp no) (fields_autoplaced)
-    (property "Reference" "D19" (at 93.98 39.0525 90)
+    (property "Reference" "D18" (at 93.98 39.0525 90)
       (effects (font (size 1.27 1.27)) (justify left))
     )
@@
       (effects (font (size 1.27 1.27)) hide)
     )
-    (pin "1")
-    (pin "2")
-    (instances
-      (project "schematic_MD"
-        (path "/3152684b-d11f-4a9a-8e6c-09965044adbd/2d267caf-42fc-44ea-97db-65c2b77a1587"
-          (reference "D19") (unit 1)
+    (property "LCSC" "C509937" (at 91.44 40.64 0)
+      (effects (font (size 1.27 1.27)) hide)
+    )
+    (property "FT Rotation Offset" "" (at 91.44 40.64 0)
+      (effects (font (size 1.27 1.27)) hide)
+    )
+    (pin "1")
+    (pin "2")
+    (instances
+      (project "schematic_MD"
+        (path "/3152684b-d11f-4a9a-8e6c-09965044adbd/2d267caf-42fc-44ea-97db-65c2b77a1587"
+          (reference "D18") (unit 1)
         )
       )
@@
     )
     (property "Datasheet" "~" (at 97.79 34.29 0)
+      (effects (font (size 1.27 1.27)) hide)
+    )
+    (property "LCSC" "C44888" (at 97.79 34.29 0)
+      (effects (font (size 1.27 1.27)) hide)
+    )
+    (property "FT Rotation Offset" "" (at 97.79 34.29 0)
       (effects (font (size 1.27 1.27)) hide)
     )
@@
       (effects (font (size 1.27 1.27)) hide)
     )
+    (property "LCSC" "C5446" (at 158.75 66.04 0)
+      (effects (font (size 1.27 1.27)) hide)
+    )
+    (property "FT Rotation Offset" "180" (at 158.75 66.04 0)
+      (effects (font (size 1.27 1.27)) hide)
+    )
     (pin "1")
     (pin "2")
@@
     )
     (property "Datasheet" "~" (at 121.92 50.8 0)
+      (effects (font (size 1.27 1.27)) hide)
+    )
+    (property "LCSC" "C51721" (at 121.92 50.8 0)
+      (effects (font (size 1.27 1.27)) hide)
+    )
+    (property "FT Rotation Offset" "" (at 121.92 50.8 0)
       (effects (font (size 1.27 1.27)) hide)
     )
@@
         )
         (path "/3152684b-d11f-4a9a-8e6c-09965044adbd/2d267caf-42fc-44ea-97db-65c2b77a1587"
-          (reference "R50") (unit 1)
+          (reference "R61") (unit 1)
         )
       )
@@
   (symbol (lib_id "Device:D_Schottky") (at 158.75 55.88 0) (unit 1)
     (in_bom yes) (on_board yes) (dnp no) (fields_autoplaced)
-    (property "Reference" "D18" (at 158.4325 49.53 0)
+    (property "Reference" "D19" (at 158.4325 49.53 0)
       (effects (font (size 1.27 1.27)))
     )
@@
       (effects (font (size 1.27 1.27)) hide)
     )
-    (pin "1")
-    (pin "2")
-    (instances
-      (project "schematic_MD"
-        (path "/3152684b-d11f-4a9a-8e6c-09965044adbd/2d267caf-42fc-44ea-97db-65c2b77a1587"
-          (reference "D18") (unit 1)
+    (property "LCSC" "C509937" (at 158.75 55.88 0)
+      (effects (font (size 1.27 1.27)) hide)
+    )
+    (property "FT Rotation Offset" "" (at 158.75 55.88 0)
+      (effects (font (size 1.27 1.27)) hide)
+    )
+    (pin "1")
+    (pin "2")
+    (instances
+      (project "schematic_MD"
+        (path "/3152684b-d11f-4a9a-8e6c-09965044adbd/2d267caf-42fc-44ea-97db-65c2b77a1587"
+          (reference "D19") (unit 1)
         )
       )
@@
       (effects (font (size 1.27 1.27)) hide)
     )
+    (property "LCSC" "C15849" (at 167.64 71.12 0)
+      (effects (font (size 1.27 1.27)) hide)
+    )
+    (property "FT Rotation Offset" "" (at 167.64 71.12 0)
+      (effects (font (size 1.27 1.27)) hide)
+    )
     (pin "1")
     (pin "2")
@@
     )
     (property "Datasheet" "~" (at 149.86 71.12 0)
+      (effects (font (size 1.27 1.27)) hide)
+    )
+    (property "LCSC" "C15849" (at 149.86 71.12 0)
+      (effects (font (size 1.27 1.27)) hide)
+    )
+    (property "FT Rotation Offset" "" (at 149.86 71.12 0)
       (effects (font (size 1.27 1.27)) hide)
     )
@@
   (symbol (lib_id "Regulator_Switching:TPS5430DDA") (at 68.58 34.29 0) (unit 1)
     (in_bom yes) (on_board yes) (dnp no) (fields_autoplaced)
-    (property "Reference" "U10" (at 68.58 21.59 0)
+    (property "Reference" "U8" (at 68.58 21.59 0)
       (effects (font (size 1.27 1.27)))
     )
@@
     )
     (property "Datasheet" "http://www.ti.com/lit/ds/symlink/tps5430.pdf" (at 68.58 34.29 0)
+      (effects (font (size 1.27 1.27)) hide)
+    )
+    (property "LCSC" "C9864" (at 68.58 34.29 0)
+      (effects (font (size 1.27 1.27)) hide)
+    )
+    (property "FT Rotation Offset" "" (at 68.58 34.29 0)
       (effects (font (size 1.27 1.27)) hide)
     )
@@
       (project "schematic_MD"
         (path "/3152684b-d11f-4a9a-8e6c-09965044adbd/2d267caf-42fc-44ea-97db-65c2b77a1587"
-          (reference "U10") (unit 1)
+          (reference "U8") (unit 1)
         )
       )
@@
   (symbol (lib_id "Device:C_Small") (at 38.1 35.56 0) (unit 1)
     (in_bom yes) (on_board yes) (dnp no)
-    (property "Reference" "C52" (at 35.56 34.2963 0)
-      (effects (font (size 1.27 1.27)) (justify right))
-    )
-    (property "Value" "10u" (at 36.83 38.1 0)
-      (effects (font (size 1.27 1.27)) (justify right))
-    )
-    (property "Footprint" "Capacitor_SMD:C_0603_1608Metric" (at 38.1 35.56 0)
+    (property "Reference" "C54" (at 35.56 34.2963 0)
+      (effects (font (size 1.27 1.27)) (justify right))
+    )
+    (property "Value" "10uF" (at 36.83 38.1 0)
+      (effects (font (size 1.27 1.27)) (justify right))
+    )
+    (property "Footprint" "Capacitor_SMD:C_0805_2012Metric" (at 38.1 35.56 0)
       (effects (font (size 1.27 1.27)) hide)
     )
@@
       (effects (font (size 1.27 1.27)) hide)
     )
-    (pin "1")
-    (pin "2")
-    (instances
-      (project "schematic_MD"
-        (path "/3152684b-d11f-4a9a-8e6c-09965044adbd/2d267caf-42fc-44ea-97db-65c2b77a1587"
-          (reference "C52") (unit 1)
+    (property "LCSC" "C440198" (at 38.1 35.56 0)
+      (effects (font (size 1.27 1.27)) hide)
+    )
+    (property "FT Rotation Offset" "" (at 38.1 35.56 0)
+      (effects (font (size 1.27 1.27)) hide)
+    )
+    (pin "1")
+    (pin "2")
+    (instances
+      (project "schematic_MD"
+        (path "/3152684b-d11f-4a9a-8e6c-09965044adbd/2d267caf-42fc-44ea-97db-65c2b77a1587"
+          (reference "C54") (unit 1)
         )
       )
@@
     )
     (property "Datasheet" "~" (at 121.92 40.64 0)
+      (effects (font (size 1.27 1.27)) hide)
+    )
+    (property "LCSC" "C25752" (at 121.92 40.64 0)
+      (effects (font (size 1.27 1.27)) hide)
+    )
+    (property "FT Rotation Offset" "" (at 121.92 40.64 0)
       (effects (font (size 1.27 1.27)) hide)
     )
@@
         )
         (path "/3152684b-d11f-4a9a-8e6c-09965044adbd/2d267caf-42fc-44ea-97db-65c2b77a1587"
-          (reference "R49") (unit 1)
-        )
-      )
+          (reference "R60") (unit 1)
+        )
+      )

Commit message: Board for ordering
Parts:
- added R4: 10k, Resistor_SMD:R_1206_3216Metric, symbol Device:R
- D18: LCSC C509937 -> C22466347
Connections:
- net 5V_OUT: now also R4.1
- net GND: now also R4.2
Other:
- moved on the sheet: C57, C58, D19, R1, U9
